File: ISA_EMS.kicad_pcb (KiCad board)
At the start: 2 copper layers, 176.5 x 85.1 mm, 49 parts, among them J1 ISA BUS, J2 EMS Address, U10 74HCT32, U11 74HCT04, U12 74LS245, U13 AS6C4008-55PCN, U14 AS6C4008-55PCN, U15 AS6C4008-55PCN, U16 AS6C4008-55PCN, U17 74HCT138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

Commit message: Reroute some traces
Routing:
- net /A14: track 144.3 -> 122.5 mm, vias 4 -> 6
Changed lines of the file:
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@@
     (thickness 1.6)
     (drawings 89)
-    (tracks 2981)
+    (tracks 2985)
     (zones 0)
     (modules 49)
@@
   )
   (module Capacitor_THT:C_Disc_D6.0mm_W2.5mm_P5.00mm (layer F.Cu)
+    (at 148.59 170.446 180)
+    (descr "C, Disc series, Radial, pin pitch=5.00mm, , diameter*width=6*2.5mm^2, Capacitor, http://cdn-reichelt.de/documents/datenblatt/B300/DS_KERKO_TC.pdf")
+    (tags "C Disc series Radial pin pitch 5.00mm  diameter 6mm width 2.5mm Capacitor")
+    (fp_text reference C18 (at -2.54 0) (layer F.SilkS)
+      (effects (font (size 1 1) (thickness 0.15)))
+    )
+    (fp_text value 100nF (at 2.5 2.5) (layer F.Fab)
+      (effects (font (size 1 1) (thickness 0.15)))
+    )
+    (fp_line (start -0.5 -1.25) (end -0.5 1.25) (layer F.Fab) (width 0.1))
+    (fp_line (start -0.5 1.25) (end 5.5 1.25) (layer F.Fab) (width 0.1))
+    (fp_line (start 5.5 1.25) (end 5.5 -1.25) (layer F.Fab) (width 0.1))
+    (fp_line (start 5.5 -1.25) (end -0.5 -1.25) (layer F.Fab) (width 0.1))
+    (fp_line (start -0.62 -1.37) (end 5.62 -1.37) (layer F.SilkS) (width 0.12))
+    (fp_line (start -0.62 1.37) (end 5.62 1.37) (layer F.SilkS) (width 0.12))
+    (fp_line (start -0.62 -1.37) (end -0.62 -0.925) (layer F.SilkS) (width 0.12))
+    (fp_line (start -0.62 0.925) (end -0.62 1.37) (layer F.SilkS) (width 0.12))
+    (fp_line (start 5.62 -1.37) (end 5.62 -0.925) (layer F.SilkS) (width 0.12))
+    (fp_line (start 5.62 0.925) (end 5.62 1.37) (layer F.SilkS) (width 0.12))
+    (fp_line (start -1.05 -1.5) (end -1.05 1.5) (layer F.CrtYd) (width 0.05))
+    (fp_line (start -1.05 1.5) (end 6.05 1.5) (layer F.CrtYd) (width 0.05))
+    (fp_line (start 6.05 1.5) (end 6.05 -1.5) (layer F.CrtYd) (width 0.05))
+    (fp_line (start 6.05 -1.5) (end -1.05 -1.5) (layer F.CrtYd) (width 0.05))
+    (fp_text user %R (at 2.5 0) (layer F.Fab)
+      (effects (font (size 1 1) (thickness 0.15)))
+    )
+    (pad 2 thru_hole circle (at 5 0 180) (size 1.6 1.6) (drill 0.8) (layers *.Cu *.Mask)
+      (net 1 GND))
+    (pad 1 thru_hole circle (at 0 0 180) (size 1.6 1.6) (drill 0.8) (layers *.Cu *.Mask)
+      (net 2 VCC))
+    (model ${KISYS3DMOD}/Capacitor_THT.3dshapes/C_Disc_D6.0mm_W2.5mm_P5.00mm.wrl
+      (at (xyz 0 0 0))
+      (scale (xyz 1 1 1))
+      (rotate (xyz 0 0 0))
+    )
+  )
+  (module Capacitor_THT:C_Disc_D6.0mm_W2.5mm_P5.00mm (layer F.Cu)
     (at 190.468 168.413 270)
     (descr "C, Disc series, Radial, pin pitch=5.00mm, , diameter*width=6*2.5mm^2, Capacitor, http://cdn-reichelt.de/documents/datenblatt/B300/DS_KERKO_TC.pdf")
@@
   )
   (module Capacitor_THT:C_Disc_D6.0mm_W2.5mm_P5.00mm (layer F.Cu)
-    (at 148.59 170.446 180)
-    (descr "C, Disc series, Radial, pin pitch=5.00mm, , diameter*width=6*2.5mm^2, Capacitor, http://cdn-reichelt.de/documents/datenblatt/B300/DS_KERKO_TC.pdf")
-    (tags "C Disc series Radial pin pitch 5.00mm  diameter 6mm width 2.5mm Capacitor")
-    (fp_text reference C18 (at -2.54 0) (layer F.SilkS)
-      (effects (font (size 1 1) (thickness 0.15)))
-    )
-    (fp_text value 100nF (at 2.5 2.5) (layer F.Fab)
-      (effects (font (size 1 1) (thickness 0.15)))
-    )
-    (fp_line (start -0.5 -1.25) (end -0.5 1.25) (layer F.Fab) (width 0.1))
-    (fp_line (start -0.5 1.25) (end 5.5 1.25) (layer F.Fab) (width 0.1))
-    (fp_line (start 5.5 1.25) (end 5.5 -1.25) (layer F.Fab) (width 0.1))
-    (fp_line (start 5.5 -1.25) (end -0.5 -1.25) (layer F.Fab) (width 0.1))
-    (fp_line (start -0.62 -1.37) (end 5.62 -1.37) (layer F.SilkS) (width 0.12))
-    (fp_line (start -0.62 1.37) (end 5.62 1.37) (layer F.SilkS) (width 0.12))
-    (fp_line (start -0.62 -1.37) (end -0.62 -0.925) (layer F.SilkS) (width 0.12))
-    (fp_line (start -0.62 0.925) (end -0.62 1.37) (layer F.SilkS) (width 0.12))
-    (fp_line (start 5.62 -1.37) (end 5.62 -0.925) (layer F.SilkS) (width 0.12))
-    (fp_line (start 5.62 0.925) (end 5.62 1.37) (layer F.SilkS) (width 0.12))
-    (fp_line (start -1.05 -1.5) (end -1.05 1.5) (layer F.CrtYd) (width 0.05))
-    (fp_line (start -1.05 1.5) (end 6.05 1.5) (layer F.CrtYd) (width 0.05))
-    (fp_line (start 6.05 1.5) (end 6.05 -1.5) (layer F.CrtYd) (width 0.05))
-    (fp_line (start 6.05 -1.5) (end -1.05 -1.5) (layer F.CrtYd) (width 0.05))
-    (fp_text user %R (at 2.5 0) (layer F.Fab)
-      (effects (font (size 1 1) (thickness 0.15)))
-    )
-    (pad 2 thru_hole circle (at 5 0 180) (size 1.6 1.6) (drill 0.8) (layers *.Cu *.Mask)
-      (net 1 GND))
-    (pad 1 thru_hole circle (at 0 0 180) (size 1.6 1.6) (drill 0.8) (layers *.Cu *.Mask)
-      (net 2 VCC))
-    (model ${KISYS3DMOD}/Capacitor_THT.3dshapes/C_Disc_D6.0mm_W2.5mm_P5.00mm.wrl
-      (at (xyz 0 0 0))
-      (scale (xyz 1 1 1))
-      (rotate (xyz 0 0 0))
-    )
-  )
-  (module Capacitor_THT:C_Disc_D6.0mm_W2.5mm_P5.00mm (layer F.Cu)
     (at 153.384 182.891 270)
     (descr "C, Disc series, Radial, pin pitch=5.00mm, , diameter*width=6*2.5mm^2, Capacitor, http://cdn-reichelt.de/documents/datenblatt/B300/DS_KERKO_TC.pdf")
@@
   (via (at 243.4959 194.3942) (size 0.8) (layers F.Cu B.Cu) (net 27))
   (segment (start 210.0516 172.7686) (end 209.0842 171.8012) (width 0.25) (layer F.Cu) (net 28))
-  (segment (start 209.0842 171.8012) (end 148.301 171.8012) (width 0.25) (layer F.Cu) (net 28))
-  (segment (start 148.301 171.8012) (end 147.4377 170.9379) (width 0.25) (layer F.Cu) (net 28))
-  (segment (start 147.4377 170.9379) (end 147.4377 169.9949) (width 0.25) (layer F.Cu) (net 28))
-  (segment (start 147.4377 169.9949) (end 151.508 165.9246) (width 0.25) (layer F.Cu) (net 28))
-  (segment (start 151.508 165.9246) (end 160.7107 165.9246) (width 0.25) (layer F.Cu) (net 28))
   (segment (start 160.7107 165.9246) (end 161.0176 165.6177) (width 0.25) (layer F.Cu) (net 28))
   (segment (start 161.0176 165.6177) (end 166.612 165.6177) (width 0.25) (layer F.Cu) (net 28))
@@
   (via (at 227.374 176.4317) (size 0.8) (layers F.Cu B.Cu) (net 28))
   (via (at 241.745 193.006) (size 0.8) (layers F.Cu B.Cu) (net 28))
+  (via (at 159.2346 170.18) (size 0.8) (drill 0.4) (layers F.Cu B.Cu) (net 28))
+  (segment (start 160.8558 171.8012) (end 159.2346 170.18) (width 0.25) (layer F.Cu) (net 28))
+  (segment (start 209.0842 171.8012) (end 160.8558 171.8012) (width 0.25) (layer F.Cu) (net 28))
+  (via (at 159.2346 166.37) (size 0.8) (drill 0.4) (layers F.Cu B.Cu) (net 28))
+  (segment (start 159.335001 170.079599) (end 159.335001 166.470401) (width 0.25) (layer B.Cu) (net 28))
+  (segment (start 159.335001 166.470401) (end 159.2346 166.37) (width 0.25) (layer B.Cu) (net 28))
+  (segment (start 159.2346 170.18) (end 159.335001 170.079599) (width 0.25) (layer B.Cu) (net 28))
+  (segment (start 159.68 165.9246) (end 160.7107 165.9246) (width 0.25) (layer F.Cu) (net 28))
+  (segment (start 159.2346 166.37) (end 159.68 165.9246) (width 0.25) (layer F.Cu) (net 28))
   (segment (start 251.46 195.2547) (end 249.5314 193.3261) (width 0.25) (layer F.Cu) (net 29))
   (segment (start 249.5314 193.3261) (end 244.498 193.3261) (width 0.25) (layer F.Cu) (net 29))

Commit message: Initial import to KiCad 7
Connections:
- net /~IOW renamed /~{IOW}
- net /~MEMR renamed /~{MEMR}
- net /~MEMW renamed /~{MEMW}
- net /~RAM-CS0 renamed /~{RAM-CS0}
- net /~RAM-CS1 renamed /~{RAM-CS1}
- net /~RAM-CS2 renamed /~{RAM-CS2}
- net /~RAM-CS3 renamed /~{RAM-CS3}
- net /~RAM-CS4 renamed /~{RAM-CS4}
- net /~RAM-CS5 renamed /~{RAM-CS5}
- net /~RAM-CS6 renamed /~{RAM-CS6}
- net /~RAM-CS7 renamed /~{RAM-CS7}
- net /~RAM-SELECT renamed /~{RAM-SELECT}
- net /~REG0-OE renamed /~{REG0-OE}
- net /~REG1-OE renamed /~{REG1-OE}
- net /~REG2-OE renamed /~{REG2-OE}
- net /~REG3-OE renamed /~{REG3-OE}
Other:
- net class Default removed
- net class POWER removed
- net class POWR_SMALL removed
